Commit message: mapeo con hectos slam

File: xacro/robot.urdf.xacro (robot description, xacro)
@@ -33,5 +33,5 @@
     <origin xyz="0 0 0.08" rpy="0 0 0"/>
   </joint>
-  <link name="wheel_right_link">
+  <link name="right_wheel">
     <visual>
       <origin xyz="0 0 0" rpy="1.57 0 0" />
@@ -48,11 +48,11 @@
     </collision>
   </link>
-  <joint name="wheel_right_joint" type="continuous">
+  <joint name="right_wheel" type="continuous">
     <parent link="base_link"/>
-    <child link="wheel_right_link"/>
+    <child link="right_wheel"/>
     <origin xyz="-0.15 0.16 -0.18" rpy="0 0 0"/> <!-- Ajusta estos valores -->
     <axis xyz="0 1 0"/>
   </joint>
-  <link name="wheel_left_link">
+  <link name="left_wheel">
     <visual>
       <origin xyz="0 0 0" rpy="-1.57 0 0" />
@@ -69,30 +69,31 @@
     </collision>
   </link>
-  <joint name="wheel_left_joint" type="continuous">
+  <joint name="left_wheel" type="continuous">
     <parent link="base_link"/>
-    <child link="wheel_left_link"/>
+    <child link="left_wheel"/>
     <origin xyz="-0.15 -0.16 -0.18" rpy="0 0 0"/> <!-- Ajusta estos valores -->
     <axis xyz="0 1 0"/>
   </joint>
-  <link name="lidar_link">
-    <visual>
-      <origin xyz="0 0 0" rpy="0 0 0"/> <!-- Sin cambios aquí -->
-      <geometry>
-        <cylinder length="0.05" radius="0.04"/> <!-- Dimensiones del LiDAR -->
-      </geometry>
-      <material name="blue"/> <!-- Color azul para el LiDAR -->
-    </visual>
-    <collision>
-      <origin xyz="0 0 0" rpy="0 0 0"/> <!-- Sin cambios aquí -->
-      <geometry>
-        <cylinder length="0.05" radius="0.04"/>
-      </geometry>
-    </collision>
-  </link>
-  <joint name="lidar_joint" type="fixed">
-    <parent link="base_link"/>
-    <child link="lidar_link"/>
-    <origin xyz="0.2 0 0.175" rpy="0 0 0"/> <!-- Centrado en el eje Y -->
-  </joint>
+  <!-- Lidar -->
+ <link name="laser">
+  <visual>
+    <origin xyz="0 0 0" rpy="0 0 0"/>
+    <geometry>
+      <cylinder length="0.05" radius="0.04"/>
+    </geometry>
+    <material name="blue"/>
+  </visual>
+  <collision>
+    <origin xyz="0 0 0" rpy="0 0 0"/>
+    <geometry>
+      <cylinder length="0.05" radius="0.04"/>
+    </geometry>
+  </collision>
+</link>
+<joint name="laser_joint" type="fixed">
+  <parent link="base_link"/>
+  <child link="laser"/>
+  <origin xyz="0.2 0 0.175" rpy="0 0 0"/>
+</joint>
   <!-- Rueda guía izquierda -->
 <link name="front_left_guide_wheel">
